Commit message: Add updated urdf and new configuration files

File: models/stickBot/model.urdf (robot description, URDF)
Before this commit: robot stickBot, 46 links, 45 joints
Links:
- added link camera_tilt, mass 0.06; visual cylinder length=0.09 radius=0.03
- added link lidar, mass 0.2; visual cylinder length=0.04 radius=0.04
- link head: geometry visual sphere radius=0.08
Joints:
- added joint camera_tilt_joint: type revolute, parent neck_3, child camera_tilt, origin xyz=0.05305 0.0 0.08205 rpy=1.5708 3.1415 0.0, axis 0 0 1.0, limit lower=-0.7853981633974483 upper=0.7853981633974483 effort=50000.0 velocity=120.0
- added joint lidar_joint: type revolute, parent neck_3, child lidar, origin xyz=0.0 0.0 0.17 rpy=0.0 0.0 0.0, axis 0 0 1.0, limit lower=-0.7853981633974483 upper=0.7853981633974483 effort=50000.0 velocity=120.0

Commit message: modify urdf for total mass as iCub3, remove Nan and continuous joint

File: models/stickBot/model.urdf (robot description, URDF)
Before this commit: robot stickBot, 48 links, 47 joints
Links:
- link base_link: mass 1.0 -> None
- link chest: mass 5.75757 -> 5.771074695
- link head: mass 1.93676 -> 1.831737118
- link imu_frame: mass 1.0 -> None
- link l_ankle_1: mass 0.366025 -> 0.3461769035
- link l_ankle_2: mass 1.06953 -> 1.011533592
- link l_elbow_1: mass 0.230254 -> 0.217768231
- link l_foot_front: mass 0.185074 -> 0.175038164
- link l_foot_rear: mass 0.184608 -> 0.174597434
- link l_forearm: mass 0.9079300000000001 -> 0.858696525
- link l_hand: mass 0.263541 -> 0.249250207
- link l_hip_1: mass 2.48546 -> 2.108461113
- link l_hip_2: mass 1.8834 -> 1.781270621
- link l_hip_3: mass 2.29352 -> 2.169151426
- link l_lower_leg: mass 5.66584 -> 5.063049414
- link l_shoulder_1: mass 1.45562 -> 1.376687449
- link l_shoulder_2: mass 0.322126 -> 0.304658373
- link l_shoulder_3: mass 0.256128 -> 0.242239185
- link l_sole: mass 1.0 -> None
- link l_upper_arm: mass 2.06334 -> 1.968325789
- link l_upper_leg: mass 2.24396 -> 0.968264435
- link l_wrist_1: mass 0.0344005 -> 0.032535096
- link neck_1: mass 0.380603 -> 0.359964395
- link neck_2: mass 0.125549 -> 0.118740971
- link neck_3: mass 0.190133 -> 0.179822835
- link r_ankle_1: mass 0.366025 -> 0.346176903
- link r_ankle_2: mass 1.06609 -> 1.00828013
- link r_elbow_1: mass 0.397478 -> 0.217609341
- link r_foot_front: mass 0.185773 -> 0.17569926
- link r_foot_rear: mass 0.184841 -> 0.174817799
- link r_forearm: mass 0.9032620000000001 -> 0.854281652
- link r_hand: mass 0.264229 -> 0.2499009
- link r_hip_1: mass 2.50002 -> 2.134290199
- link r_hip_2: mass 1.881 -> 1.779000764
- link r_hip_3: mass 2.29213 -> 2.1678368
- link r_lower_leg: mass 5.898710000000001 -> 5.074105512
- link r_shoulder_1: mass 1.45988 -> 1.380716446
- link r_shoulder_2: mass 0.322126 -> 0.304658373
- link r_shoulder_3: mass 0.258699 -> 0.24467077
- link r_sole: mass 1.0 -> None
- link r_upper_arm: mass 2.06334 -> 1.960447492
- link r_upper_leg: mass 2.2571 -> 0.980691904
- link r_wrist_1: mass 0.0344005 -> 0.032535096
- link root_link: mass 2.67135 -> 2.52649319
- link torso_1: mass 1.81255 -> 1.714262538
- link torso_2: mass 1.45349 -> 1.374672951
Joints:
- joint base_link_fixed_joint: axis nan nan nan -> 0 0 0
- joint camera_tilt_joint: axis 0 0 1.0 -> 0. 0. 1.; origin xyz=0.05305 0.0 0.08205 rpy=1.5708 3.1415 0.0 -> xyz=0.05305 0.0 0.08205 rpy=-1.5707926535897934 9.265358979305728e-05 -3.141592653589793
- joint l_hip_pitch: origin xyz=0.0216 0.04045000000000001 0.0 rpy=0.0 0.0 0.0 -> xyz=0.0216 0.04045000000000001 -0.021599999999999994 rpy=0.0 0.0 0.0
- joint l_shoulder_pitch: origin xyz=-0.03 0.055555 0.16 rpy=0.25326164431680925 0.0 -0.26179970938509745 -> xyz=-0.03 0.055555 0.163 rpy=0.25326164431680925 0.0 -0.26179970938509745
- joint lidar_joint: axis 0 0 1.0 -> 0. 0. 1.
- joint neck_fixed_joint: origin xyz=-0.00378849 0.0 0.1652995 rpy=0.0 0.0 0.0 -> xyz=-0.00378849 0.0 0.1683 rpy=0.0 0.0 0.0
- joint r_hip_pitch: origin xyz=0.0216 -0.040549999999999996 0.0 rpy=0.0 0.0 0.0 -> xyz=0.0216 -0.040549999999999996 -0.021599999999999994 rpy=0.0 0.0 0.0
- joint r_shoulder_pitch: origin xyz=-0.03 -0.055555 0.16 rpy=-0.25326164431680925 0.0 0.26179970938509745 -> xyz=-0.03 -0.055555 0.163 rpy=-0.25326164431680925 0.0 0.26179970938509745
- joint r_wrist_yaw: limit (none) -> lower=-0.2617993877991494 upper=0.6108652381980153 effort=50000.0 velocity=120.0; type continuous -> revolute
- joint torso_pitch: origin xyz=0.0 0.0 0.07250000000000001 rpy=0.0 0.0 0.0 -> xyz=0.0 0.0 0.0725 rpy=0.0 0.0 0.0
- joint torso_yaw: origin xyz=0.0 0.0 0.06447000000000001 rpy=0.0 0.0 0.0 -> xyz=0.0 0.0 0.06447 rpy=0.0 0.0 0.0

Commit message: fix wrong origins

File: models/stickBot/model.urdf (robot description, URDF)
Before this commit: robot stickBot, 48 links, 47 joints
Joints:
- joint camera_tilt_joint: origin xyz=0.05305 0.0 0.08205 rpy=-1.5707926535897934 9.265358979305728e-05 -3.141592653589793 -> xyz=0.05305 0.0 0.08205 rpy=1.5708 3.1415 0.0
- joint l_hip_pitch: origin xyz=0.0216 0.04045000000000001 -0.021599999999999994 rpy=0.0 0.0 0.0 -> xyz=0.0216 0.04045000000000001 0.0 rpy=0.0 0.0 0.0
- joint r_hip_pitch: origin xyz=0.0216 -0.040549999999999996 -0.021599999999999994 rpy=0.0 0.0 0.0 -> xyz=0.0216 -0.040549999999999996 0.0 rpy=0.0 0.0 0.0

Commit message: added collision on feet

File: models/stickBot/model.urdf (robot description, URDF)
Before this commit: robot stickBot, 48 links, 47 joints
Links:
- link l_foot_front: geometry collision box size=0.1 0.117 0.0103; visual box size=0.1 0.117 0.0103
- link l_foot_rear: geometry collision box size=0.1 0.117 0.0103; visual box size=0.1 0.117 0.0103
- link r_foot_front: geometry collision box size=0.1 0.117 0.0103; visual box size=0.1 0.117 0.0103
- link r_foot_rear: geometry collision box size=0.1 0.117 0.0103; visual box size=0.1 0.117 0.0103

Commit message: aggiunti file per esporre su ROS i topic di lidar, camera e joint_states

File: models/stickBot/model.urdf (robot description, URDF)
Before this commit: robot stickBot, 48 links, 47 joints
Joints:
- joint lidar_joint: type revolute -> fixed

Commit message: update Lidar and camera joints frame origins and replace parent link with head and not neck_3

File: models/stickBot/model.urdf (robot description, URDF)
Before this commit: robot stickBot, 48 links, 47 joints
Joints:
- joint camera_tilt_joint: origin xyz=0.05305 0.0 0.08205 rpy=1.5708 3.1415 0.0 -> xyz=0.055513 0.00017 0.076925 rpy=1.5708 3.1415 0.0; parent neck_3 -> head
- joint lidar_joint: origin xyz=0.0 0.0 0.17 rpy=0.0 0.0 0.0 -> xyz=0.00117 0.00115 0.1268 rpy=0.0 0.0 0.0; parent neck_3 -> head
